File: bldc_controller/bldc_controller.sch (KiCad schematic (older format))
At the start: 84 parts

Commit message: Partially linked footprints to symbols
Parts:
- removed C?: 100n, symbol bldc_controller-rescue:C_Small-Device
- removed C? (x3): 0.1u, symbol bldc_controller-rescue:C-Device
- removed IC?: mcp6004-e_p, DIP781W56P254L1918H533Q14N, symbol bldc_controller-rescue:mcp6004-e_p-mcp6004-e_p
- removed IC? (x3): ACS37002LMABTR-066B3, SOIC127P1030X265-16N, symbol bldc_controller-rescue:ACS37002LMABTR-066B3-ACS37002LMABTR-066B3
- added C17, C33, C34, C35: C-Device, symbol bldc_controller-rescue:C-Device
- added IC5, IC6, IC7: ACS712ELCTR-30A-T, ACS712ELCTR-30A-T:SOIC127P600X175-8N, symbol ACS712ELCTR-30A-T:ACS712ELCTR-30A-T
- added PS1: TSR_1-48150WI, symbol bldc_controller-rescue:TSR_1-48150WI-TSR_1-48150WI
- added PS2: TSR_0.6-4850WI, symbol bldc_controller-rescue:TSR_0.6-4850WI-TSR_0.6-4850WI
- IC1: renamed from IC?; footprint TO255P460X1020X2008-3P -> (none)
- IC2, IC3, IC4: renamed from IC?; footprint DIP762W56P254L988H533Q8N -> (none)
- J2: renamed from J?; symbol Connector:Conn_01x03_Male -> bldc_controller-rescue:Conn_01x03_Male-Connector
- PS3: renamed from PS?; footprint R78HB3305L -> (none)
- R10, R11, R12, R13, R8, R9: renamed from R?; value 4.7 -> 1.5
- gave numbers to parts that had none: 64
Connections:
- net +48V: now also PS1.1 (+VIN)
- net A_CURR_VOUT: now also IC5.7 (VIOUT)
- net BUCK_IN: now also C17.1, PS2.1 (+VIN)
- net B_CURR_VOUT: now also IC6.7 (VIOUT)
- net C_CURR_VOUT: now also IC7.7 (VIOUT)
- net DRIVE_VCC: now also PS1.3 (+VOUT)
- net GND: now also C17.2, C33.2, C34.2, C35.2, IC5.5 (GND), IC6.5 (GND), IC7.5 (GND), PS1.2 (GND), PS1.4 (CASE_PIN_1), PS1.5 (CASE_PIN_2), PS2.2 (GND)
- net MOT_A: now also IC5.3 (IP-_1), IC5.4 (IP-_2)
- net MOT_B: now also IC6.3 (IP-_1), IC6.4 (IP-_2)
- net MOT_C: now also IC7.3 (IP-_1), IC7.4 (IP-_2)
- net VOUT_A: now also IC5.1 (IP+_1), IC5.2 (IP+_2)
- net VOUT_B: now also IC6.1 (IP+_1), IC6.2 (IP+_2)
- net VOUT_C: now also IC7.1 (IP+_1), IC7.2 (IP+_2)
- new net: C33.1, IC5.6 (FILTER)
- new net: C34.1, IC6.6 (FILTER)
- new net: C35.1, IC7.6 (FILTER)
- new net 5V_BAT: IC5.8 (VCC), IC6.8 (VCC), IC7.8 (VCC), PS2.3 (+VOUT)
Other:
- note removed: "Note - these need to go to ADC pins"
- moved on the sheet: C23, C24, C25, C26, C27, C31, C32, IC1, PS3, R14, R15, R16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
