File: bldc_controller/bldc_controller.kicad_sch (KiCad schematic)
At the start: 85 parts, among them IC1 LF33CV, IC2 IRS2003PBF, IC3 IRS2003PBF, IC4 IRS2003PBF, IC5 ACS712ELCTR-30A-T, IC6 ACS712ELCTR-30A-T, IC7 ACS712ELCTR-30A-T, J1 Screw_Terminal_01x02, J2 Conn_01x03_Male, J3 USB_B_Micro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

Commit message: Worked on footprints
Parts:
- removed Q2, Q3, Q4, Q5, Q6, Q7: Q_NMOS_GSD, symbol bldc_controller-rescue:Q_NMOS_GSD-Device
- added Q2, Q3, Q4, Q5, Q6, Q7: TK72E12N1,S1X_S, TK72E12N1,S1X_S:TO254P465X1016X1935-3P, symbol TK72E12N1_S1X_S:TK72E12N1,S1X_S
- C1: footprint Capacitor_SMD:C_0603_1608Metric -> LED_SMD:LED_1206_3216Metric
- C17, C23: value C-Device -> 1u; footprint (none) -> Capacitor_SMD:C_0603_1608Metric
- C33, C34, C35: value C-Device -> 1n; footprint (none) -> Capacitor_SMD:C_0603_1608Metric
- D1: footprint (none) -> LED_SMD:LED_1206_3216Metric
- D2, D3, D4: footprint (none) -> Diode_THT:D_DO-41_SOD81_P10.16mm_Horizontal
- F1: footprint (none) -> Fuse:Fuse_0805_2012Metric
- FB1: footprint (none) -> Resistor_SMD:R_0603_1608Metric
- Q1: footprint (none) -> Package_TO_SOT_THT:TO-220-3_Horizontal_TabDown
- R3: value 1k5 -> 30R
Connections:
- net +48V: now also Q2.2, Q4.2, Q6.2
- net GATE_AH: now also Q2.1
- net GATE_AL: now also Q3.1
- net GATE_BH: now also Q4.1
- net GATE_BL: now also Q5.1
- net GATE_CH: now also Q6.1
- net GATE_CL: now also Q7.1
- net GND: now also Q3.3, Q5.3, Q7.3
- net VOUT_A: now also Q2.3, Q3.2
- net VOUT_B: now also Q4.3, Q5.2
- net VOUT_C: now also Q6.3, Q7.2

Commit message: Finished footprint assignment
Note: need to choose screw terminals for motor and battery connections. Need max. current/voltage and cable gauge to choose.
Parts:
- J2: footprint (none) -> Connector_PinHeader_2.54mm:PinHeader_1x03_P2.54mm_Vertical
- J3: footprint (none) -> Connector_USB:USB_Micro-B_Molex-105017-0001
- J4: footprint (none) -> Connector_PinHeader_2.54mm:PinHeader_2x05_P2.54mm_Vertical
- L1: footprint (none) -> Inductor_SMD:L_0603_1608Metric
- PS1: footprint (none) -> TSR_1-48150:NE555DR
- PS2: footprint (none) -> TSR_0:TSR064850WI
- PS3: footprint (none) -> R-78HB3.3-0:R78HB3305
- SW1: footprint (none) -> Button_Switch_THT:SW_E-Switch_EG1271_DPDT
- Y1: footprint (none) -> Crystal:Crystal_SMD_3225-4Pin_3.2x2.5mm
